File: transmitter.sch (KiCad schematic (older format))
At the start: 0 parts

Commit message: Added transmitter
Parts:
- added C? (x7): 100p, symbol Device:C_Small
- added C? (x6): 2.2u, symbol Device:C_Small
- added J? (x2): Conn_Coaxial, symbol Connector:Conn_Coaxial
- added R?: 49.9, symbol Device:R
- added R? (x2): 0, symbol Device:R
- added R? (x5): DNP, symbol Device:R
- added R?: 52.3, symbol Device:R
- added R? (x2): 115, symbol Device:R
- added R? (x2): 10k, symbol Device:R
- added U?: HMC430, Package_DFN_QFN:QFN-24-1EP_4x4mm_P0.5mm_EP2.6x2.6mm, symbol own:HMC430
- added U?: RFPA5542, Package_DFN_QFN:QFN-20-1EP_4x4mm_P0.5mm_EP2.5x2.5mm, symbol own:RFPA5542
- added U? (x2): Opamp_Dual_Generic, symbol Device:Opamp_Dual_Generic
- added Z?: Coupler_13dB, own:Coupler_13dB, symbol own:Coupler_13dB
Connections:
- new net: R?.1, R?.2, U?.16 (RFOUT)
- new net: R?.1, R?.1, U?.1, U?.22 (VTUNE)
- new net: R?.2, Z?.4
- new net: C?.1, U?.13 (RF_OUT)
- new net: C?.2, R?.1, Z?.1
- new net: C?.1, R?.1, U?.10 (PDET)
- new net: C?.1, R?.1, R?.2, U?.5 (PA_EN)
- new net: C?.2, U?.3 (RF_IN)
- new net: C?.1, R?.1, R?.1, R?.1
- new net: R?.1, R?.2, U?.2 (-)
- new net: J?.1 (In), R?.2 (x2)
- new net +10V: C?.2, U?.8 (V+)
- new net +3V3: C?.1, C?.1, U?.20 (Vcc)
- new net +5V: C?.1, C?.1, C?.1, C?.1, C?.1, C?.1, R?.1, U?.18 (VCC3), U?.19 (VCC2), U?.20 (VCC1)
- new net GND: C?.1, C?.2, C?.2, C?.2, C?.2, C?.2, C?.2, C?.2, C?.2, C?.2, C?.2, J?.2 (Ext), J?.2 (Ext), R?.1, R?.2, R?.2, R?.2, R?.2, U?.11 (GND), U?.12 (GND), U?.14 (GND), U?.15 (GND), U?.15 (GND), U?.16 (GND), U?.17 (GND), U?.2 (GND), U?.21 (GND), U?.26 (GND), U?.4 (GND), U?.4 (V-)
- new net LO_OUT: Z?.3
- new net PA_EN: R?.2
- new net PDET: R?.1, R?.2
- new net RF_OUT: Z?.2
- new net VCO_TUNE_IN: R?.2, U?.3 (+)
Other:
- note added: "-6dBm"
- note added: "0-5V, change gain\nif different input range"
- note added: "14dBm"
- note added: "26dBm\n"
- note added: "27dBm"
- note added: "2dBm"
- note added: "Add negative supply\nif not rail to rail"
- note added: "MAYBE 3V?\n"
