File: transmitter.sch (KiCad schematic (older format))
At the start: 26 parts, among them J10 Conn_Coaxial, J9 Conn_Coaxial, U23 HMC430, U24 RFPA5542

Commit message: IF and power layout mostly finished
Parts:
- J10, J9: footprint Connector_Coaxial:SMA_Amphenol_901-144_Vertical -> Connector_Coaxial:SMA_Amphenol_132134-11_Vertical
Changed lines of the file:
@@
 F 0 "J10" V 8250 4550 50  0000 L CNN
 F 1 "Conn_Coaxial" V 8350 4300 50  0000 L CNN
-F 2 "Connector_Coaxial:SMA_Amphenol_901-144_Vertical" H 8250 4400 50  0001 C CNN
+F 2 "Connector_Coaxial:SMA_Amphenol_132134-11_Vertical" H 8250 4400 50  0001 C CNN
 F 3 " ~" H 8250 4400 50  0001 C CNN
 	1    8250 4400
@@
 F 0 "J9" V 5750 3250 50  0000 L CNN
 F 1 "Conn_Coaxial" V 5650 3050 50  0000 L CNN
-F 2 "Connector_Coaxial:SMA_Amphenol_901-144_Vertical" H 5550 3300 50  0001 C CNN
+F 2 "Connector_Coaxial:SMA_Amphenol_132134-11_Vertical" H 5550 3300 50  0001 C CNN
 F 3 " ~" H 5550 3300 50  0001 C CNN
 	1    5550 3300

Commit message: Added names
Parts:
- C55, C57, C61: footprint Capacitor_SMD:C_0603_1608Metric_Pad1.08x0.95mm_HandSolder -> Resistor_SMD:R_0402_1005Metric_Pad0.72x0.64mm_HandSolder
Changed lines of the file:
@@
 F 0 "C55" V 7000 3050 50  0000 L CNN
 F 1 "100pF" V 6900 3000 50  0000 L CNN
-F 2 "Capacitor_SMD:C_0603_1608Metric_Pad1.08x0.95mm_HandSolder" H 6800 3100 50  0001 C CNN
+F 2 "Resistor_SMD:R_0402_1005Metric_Pad0.72x0.64mm_HandSolder" H 6800 3100 50  0001 C CNN
 F 3 "~" H 6800 3100 50  0001 C CNN
 	1    6800 3100
@@
 F 0 "C57" V 7700 3050 50  0000 L CNN
 F 1 "100pF" V 7600 3000 50  0000 L CNN
-F 2 "Capacitor_SMD:C_0603_1608Metric_Pad1.08x0.95mm_HandSolder" H 7500 3100 50  0001 C CNN
+F 2 "Resistor_SMD:R_0402_1005Metric_Pad0.72x0.64mm_HandSolder" H 7500 3100 50  0001 C CNN
 F 3 "~" H 7500 3100 50  0001 C CNN
 	1    7500 3100
@@
 F 0 "C61" V 8350 3050 50  0000 L CNN
 F 1 "100pF" V 8250 3000 50  0000 L CNN
-F 2 "Capacitor_SMD:C_0603_1608Metric_Pad1.08x0.95mm_HandSolder" H 8150 3100 50  0001 C CNN
+F 2 "Resistor_SMD:R_0402_1005Metric_Pad0.72x0.64mm_HandSolder" H 8150 3100 50  0001 C CNN
 F 3 "~" H 8150 3100 50  0001 C CNN
 	1    8150 3100
