File: receiver_rf.sch (KiCad schematic (older format))
At the start: 28 parts, among them J6 Conn_Coaxial, J7 Conn_Coaxial, J8 Conn_Coaxial, U13 PMA-63GLN+, U14 RFSW8008, U15 PMA-63GLN+, U16 RFSW8008, U17 HMC218BMS8GE

Commit message: -2.5V regulator footprint added. RF switch footprint created and added.
Parts:
- U14, U16: footprint (none) -> own:QFN_7_RFSW8008
Changed lines of the file:
@@
 F 0 "U14" H 4475 4027 50  0000 C CNN
 F 1 "RFSW8008" H 4475 3936 50  0000 C CNN
-F 2 "" H 4200 4750 50  0001 C CNN
+F 2 "own:QFN_7_RFSW8008" H 4200 4750 50  0001 C CNN
 F 3 "" H 4200 4750 50  0001 C CNN
 	1    4400 4300
@@
 F 0 "U16" H 7925 3927 50  0000 C CNN
 F 1 "RFSW8008" H 7925 3836 50  0000 C CNN
-F 2 "" H 7650 4650 50  0001 C CNN
+F 2 "own:QFN_7_RFSW8008" H 7650 4650 50  0001 C CNN
 F 3 "" H 7650 4650 50  0001 C CNN
 	1    7850 4200

Commit message: First layout
Parts:
- removed U14, U16: RFSW8008, own:QFN_7_RFSW8008, symbol own:RFSW8008
- added C47, C48: 100n, Capacitor_SMD:C_0603_1608Metric_Pad1.08x0.95mm_HandSolder, symbol Device:C
- added U14, U16: QPC6324, Package_DFN_QFN:QFN-20-1EP_4x4mm_P0.5mm_EP2.5x2.5mm, symbol own:QPC6324
- C27, C33: value 82pF -> 220pF
- C32: footprint Capacitor_SMD:C_0402_1005Metric_Pad0.74x0.62mm_HandSolder -> Capacitor_SMD:C_0402_1005Metric
- J6, J7, J8: footprint (none) -> Connector_Coaxial:SMA_Amphenol_901-144_Vertical
Connections:
- net +5V: now also C47.1, C48.1, U14.20 (VDD), U16.20 (VDD)
- net GND: now also C47.2, C48.2, U14.1 (GND), U14.10 (GND), U14.11 (GND), U14.12 (GND), U14.14 (GND), U14.15 (GND), U14.18 (GND), U14.19 (GND), U14.2 (GND), U14.4 (GND), U14.5 (GND), U14.6 (GND), U14.7 (GND), U14.9 (GND), U16.1 (GND), U16.10 (GND), U16.11 (GND), U16.12 (GND), U16.14 (GND), U16.15 (GND), U16.18 (GND), U16.19 (GND), U16.2 (GND), U16.4 (GND), U16.5 (GND), U16.6 (GND), U16.7 (GND), U16.9 (GND)
- net SW_CTR1: now also C26.2, U14.17 (CTR1), U16.16 (CTR2); no longer C27.1
- net SW_CTR2: now also C27.1, U14.16 (CTR2), U16.17 (CTR1); no longer C26.2
- net at C35.1, C36.1: now also U16.8 (RFC)
- net at C25.2: now also U14.8 (RFC)
- net at C28.1: now also U14.3 (RF1)
- net at C29.1: now also U14.13 (RF2)
- net at C32.2: now also U16.13 (RF2)
- net at C29.2: now also U16.3 (RF1)
Other:
- note removed: "Control voltage 1.8V"
- moved on the sheet: C26, C33, C34, J7

Commit message: Curved tracks
Parts:
- removed C24, C35, C38: DNP, Capacitor_SMD:C_0402_1005Metric, symbol Device:C
- removed C25, C36, C37: 100pF, Capacitor_SMD:C_0402_1005Metric, symbol Device:C
- added CJ1, CJ2, CJ3: 100pF, own:0402_Jumper_Tapered, symbol own:C_Jumper
- C21, C28, C29, C32: footprint Capacitor_SMD:C_0402_1005Metric -> own:0402_Tapered
Connections:
- net LO_IN: now also CJ3.1
- net at U16.8 (RFC): now also CJ2.1
- net at U17.8 (RF): now also CJ2.2
- net at L1.2, U13.8 (RF_OUT/DC_IN): now also CJ1.1
- net at U17.1 (LO): now also CJ3.2
- net at J6.1 (In): now also CJ1.3
- net at U14.8 (RFC): now also CJ1.2
- net at J7.1 (In): now also CJ2.3
- net at J8.1 (In): now also CJ3.3
Changed lines of the file:
@@
 F 0 "C21" V 998 4400 50  0000 C CNN
 F 1 "100pF" V 1089 4400 50  0000 C CNN
-F 2 "Capacitor_SMD:C_0402_1005Metric" H 1288 4250 50  0001 C CNN
+F 2 "own:0402_Tapered" H 1288 4250 50  0001 C CNN
 F 3 "~" H 1250 4400 50  0001 C CNN
 	1    1250 4400
@@
 Wire Wire Line
 	1100 4400 1050 4400
-$Comp
-L Device:C C36
-U 1 1 5F8B8D04
-P 8950 4200
-F 0 "C36" V 8698 4200 50  0000 C CNN
-F 1 "100pF" V 8789 4200 50  0000 C CNN
-F 2 "Capacitor_SMD:C_0402_1005Metric" H 8988 4050 50  0001 C CNN
-F 3 "~" H 8950 4200 50  0001 C CNN
-	1    8950 4200
-	0    -1   1    0
-$EndComp
 Wire Wire Line
 	2900 4300 3100 4300
@@
 Text Notes 10850 4850 2    50   ~ 0
 Conversion Loss: -7dB\nP1dB: 10dB
-$Comp
-L Device:C C24
-U 1 1 5FA1A18D
-P 3550 4100
-F 0 "C24" V 3298 4100 50  0000 C CNN
-F 1 "DNP" V 3389 4100 50  0000 C CNN
-F 2 "Capacitor_SMD:C_0402_1005Metric" H 3588 3950 50  0001 C CNN
-F 3 "~" H 3550 4100 50  0001 C CNN
-	1    3550 4100
-	1    0    0    1
-$EndComp
 $Comp
 L Connector:Conn_Coaxial J6
@@
 $EndComp
 $Comp
-L Device:C C25
-U 1 1 60441535
-P 3750 4300
-F 0 "C25" V 3498 4300 50  0000 C CNN
-F 1 "100pF" V 3589 4300 50  0000 C CNN
-F 2 "Capacitor_SMD:C_0402_1005Metric" H 3788 4150 50  0001 C CNN
-F 3 "~" H 3750 4300 50  0001 C CNN
-	1    3750 4300
-	0    -1   1    0
-$EndComp
-Wire Wire Line
-	3900 4300 4050 4300
-$Comp
 L Device:C C28
 U 1 1 604497EA
@@
 F 0 "C28" V 4898 4200 50  0000 C CNN
 F 1 "100pF" V 4989 4200 50  0000 C CNN
-F 2 "Capacitor_SMD:C_0402_1005Metric" H 5188 4050 50  0001 C CNN
+F 2 "own:0402_Tapered" H 5188 4050 50  0001 C CNN
 F 3 "~" H 5150 4200 50  0001 C CNN
 	1    5150 4200
@@
 F 0 "C32" V 6848 4100 50  0000 C CNN
 F 1 "100pF" V 6939 4100 50  0000 C CNN
-F 2 "Capacitor_SMD:C_0402_1005Metric" H 7138 3950 50  0001 C CNN
+F 2 "own:0402_Tapered" H 7138 3950 50  0001 C CNN
 F 3 "~" H 7100 4100 50  0001 C CNN
 	1    7100 4100
@@
 Wire Wire Line
 	6850 4100 6900 4100
-Wire Wire Line
-	9100 4200 9150 4200
 Wire Wire Line
 	4900 4400 4950 4400
@@
 	6900 4100 6950 4100
 Wire Wire Line
-	3600 4300 3550 4300
-Connection ~ 3100 4300
-Wire Wire Line
-	3550 4250 3550 4300
-Connection ~ 3550 4300
-Wire Wire Line
-	3550 4300 3100 4300
-Wire Wire Line
 	3300 3650 3300 3600
 Wire Wire Line
 	3300 3600 3350 3600
-Wire Wire Line
-	3550 3800 3550 3950
 Wire Wire Line
 	9100 3850 9150 3850
@@
 Text HLabel 7750 2200 1    50   Input ~ 0
 SW_CTR1
-$Comp
-L Device:C C35
-U 1 1 6054EDB0
-P 8750 4000
-F 0 "C35" V 8498 4000 50  0000 C CNN
-F 1 "DNP" V 8589 4000 50  0000 C CNN
-F 2 "Capacitor_SMD:C_0402_1005Metric" H 8788 3850 50  0001 C CNN
-F 3 "~" H 8750 4000 50  0001 C CNN
-	1    8750 4000
-	1    0    0    1
-$EndComp
 $Comp
 L Connector:Conn_Coaxial J7
@@
 Wire Wire Line
 	8600 3500 8650 3500
-Wire Wire Line
-	8800 4200 8750 4200
-Wire Wire Line
-	8750 4150 8750 4200
-Connection ~ 8750 4200
-Wire Wire Line
-	8750 4200 8300 4200
 Text Notes 5850 3900 2    50   ~ 0
 1.8-6.0GHz\nNF: 1dB\nGain: +26dB\nP1dB: 11dB
-$Comp
-L Device:C C38
-U 1 1 6089D7FB
-P 9300 3000
-F 0 "C38" V 9048 3000 50  0000 C CNN
-F 1 "DNP" V 9139 3000 50  0000 C CNN
-F 2 "Capacitor_SMD:C_0402_1005Metric" H 9338 2850 50  0001 C CNN
-F 3 "~" H 9300 3000 50  0001 C CNN
-	1    9300 3000
-	0    -1   1    0
-$EndComp
 $Comp
 L Connector:Conn_Coaxial J8
@@
 Wire Wire Line
 	9800 3250 9800 3200
-Wire Wire Line
-	9600 3000 9450 3000
-Wire Wire Line
-	9100 3300 9100 3000
-Wire Wire Line
-	9150 3000 9100 3000
-Connection ~ 9100 3000
-Wire Wire Line
-	9100 2400 9100 3000
-Wire Wire Line
-	9100 3600 9100 3850
-$Comp
-L Device:C C37
-U 1 1 6089D7F5
-P 9100 3450
-F 0 "C37" V 8848 3450 50  0000 C CNN
-F 1 "100pF" V 8939 3450 50  0000 C CNN
-F 2 "Capacitor_SMD:C_0402_1005Metric" H 9138 3300 50  0001 C CNN
-F 3 "~" H 9100 3450 50  0001 C CNN
-	1    9100 3450
-	-1   0    0    -1
-$EndComp
 $Comp
 L power:GND #PWR044
@@
 F 0 "C29" V 5848 4900 50  0000 C CNN
 F 1 "100pF" V 5939 4900 50  0000 C CNN
-F 2 "Capacitor_SMD:C_0402_1005Metric" H 6138 4750 50  0001 C CNN
+F 2 "own:0402_Tapered" H 6138 4750 50  0001 C CNN
 F 3 "~" H 6100 4900 50  0001 C CNN
 	1    6100 4900
@@
 Wire Wire Line
 	8850 3800 8750 3800
-Wire Wire Line
-	8750 3800 8750 3850
 $Comp
 L power:GND #PWR0105
@@
 	-1   0    0    -1
 $EndComp
+Wire Wire Line
+	3100 4300 3400 4300
+Connection ~ 3100 4300
+Wire Wire Line
+	3850 4300 4050 4300
+Wire Wire Line
+	3550 3800 3550 4000
+$Comp
+L own:C_Jumper CJ1
+U 1 1 606940F6
+P 3550 4150
+F 0 "CJ1" H 3625 3841 50  0000 C CNN
+F 1 "100pF" H 3625 3750 50  0000 C CNN
+F 2 "own:0402_Jumper_Tapered" H 3588 4000 50  0001 C CNN
+F 3 "~" H 3550 4150 50  0001 C CNN
+	1    3550 4150
+	1    0    0    -1
+$EndComp
+$Comp
+L own:C_Jumper CJ2
+U 1 1 60694762
+P 8750 4050
+F 0 "CJ2" H 8825 3741 50  0000 C CNN
+F 1 "100pF" H 8825 3650 50  0000 C CNN
+F 2 "own:0402_Jumper_Tapered" H 8788 3900 50  0001 C CNN
+F 3 "~" H 8750 4050 50  0001 C CNN
+	1    8750 4050
+	1    0    0    -1
+$EndComp
+Wire Wire Line
+	8750 3800 8750 3900
+Wire Wire Line
+	9050 4200 9150 4200
+Wire Wire Line
+	8600 4200 8300 4200
+$Comp
+L own:C_Jumper CJ3
+U 1 1 606A173C
+P 9250 3000
+F 0 "CJ3" V 9279 2735 50  0000 R CNN
+F 1 "100pF" V 9370 2735 50  0000 R CNN
+F 2 "own:0402_Jumper_Tapered" H 9288 2850 50  0001 C CNN
+F 3 "~" H 9250 3000 50  0001 C CNN
+	1    9250 3000
+	0    1    1    0
+$EndComp
+Wire Wire Line
+	9400 3000 9600 3000
+Wire Wire Line
+	9100 2850 9100 2400
+Wire Wire Line
+	9100 3300 9100 3850
 $EndSCHEMATC
