File: Radar.sch (KiCad schematic (older format))
At the start: 13 parts, among them J1 Receive_Antenna, J2 VCO_Tune, J3 Transmit Antenna, J4 Output, U1 LNA_1, U2 SW1, U3 LNA_2, U4 VCO, U5 SW2, U6 PA, U7 mixer_diagram, U8 PGA, U9 lowpass_diagram

Commit message: Added RX shield
Parts:
- J1, J2, J3, J4: footprint own:SMA_ADAM_TECH_edge_mount -> own:SMA_ADAM_TECH_edge
Changed lines of the file:
@@
 F 0 "J3" H 7550 2925 50  0000 L CNN
 F 1 "Transmit Antenna" H 7050 3100 50  0000 L CNN
-F 2 "own:SMA_ADAM_TECH_edge_mount" H 7450 2950 50  0001 C CNN
+F 2 "own:SMA_ADAM_TECH_edge" H 7450 2950 50  0001 C CNN
 F 3 " ~" H 7450 2950 50  0001 C CNN
 	1    7450 2950
@@
 F 0 "J1" H 2550 4825 50  0000 L CNN
 F 1 "Receive_Antenna" H 2050 5000 50  0000 L CNN
-F 2 "own:SMA_ADAM_TECH_edge_mount" H 2450 4850 50  0001 C CNN
+F 2 "own:SMA_ADAM_TECH_edge" H 2450 4850 50  0001 C CNN
 F 3 " ~" H 2450 4850 50  0001 C CNN
 	1    2450 4850
@@
 F 0 "J4" H 9900 4825 50  0000 L CNN
 F 1 "Output" H 9650 5000 50  0000 L CNN
-F 2 "own:SMA_ADAM_TECH_edge_mount" H 9800 4850 50  0001 C CNN
+F 2 "own:SMA_ADAM_TECH_edge" H 9800 4850 50  0001 C CNN
 F 3 " ~" H 9800 4850 50  0001 C CNN
 	1    9800 4850
@@
 F 0 "J2" H 3950 2925 50  0000 L CNN
 F 1 "VCO_Tune" H 3700 3100 50  0000 L CNN
-F 2 "own:SMA_ADAM_TECH_edge_mount" H 3850 2950 50  0001 C CNN
+F 2 "own:SMA_ADAM_TECH_edge" H 3850 2950 50  0001 C CNN
 F 3 " ~" H 3850 2950 50  0001 C CNN
 	1    3850 2950
