File: receiver_if.sch (KiCad schematic (older format))
At the start: 0 parts

Commit message: Architecture of IF
Parts:
- added C? (x7): C, symbol Device:C
- added R? (x13): R, symbol Device:R
- added U? (x5): Opamp_Dual_Generic, symbol Device:Opamp_Dual_Generic
- added U?: MCP4018-xxxxLT, Package_TO_SOT_SMD:SOT-363_SC-70-6, symbol Potentiometer_Digital:MCP4018-xxxxLT
Connections:
- net labels added: GND, IF_IN, IF_OUT
- wire segments 0 -> 66
Other:
- note added: "Add buffer to match impedance?"

Commit message: Finished IF
Parts:
- removed C? (x6): C, symbol Device:C
- removed R? (x11): R, symbol Device:R
- removed U? (x5): Opamp_Dual_Generic, symbol Device:Opamp_Dual_Generic
- removed U?: MCP4018-xxxxLT, Package_TO_SOT_SMD:SOT-363_SC-70-6, symbol Potentiometer_Digital:MCP4018-xxxxLT
- added C1, C4: 1uF, Capacitor_SMD:C_0603_1608Metric_Pad1.08x0.95mm_HandSolder, symbol Device:C
- added C10, C9: 10uF, Capacitor_SMD:C_0603_1608Metric_Pad1.08x0.95mm_HandSolder, symbol Device:C
- added C11: 51pF, Capacitor_SMD:C_0603_1608Metric_Pad1.08x0.95mm_HandSolder, symbol Device:C
- added C12, C6: 10pF, Capacitor_SMD:C_0603_1608Metric_Pad1.08x0.95mm_HandSolder, symbol Device:C
- added C13, C14, C17, C18: 1nF, Capacitor_SMD:C_0603_1608Metric_Pad1.08x0.95mm_HandSolder, symbol Device:C
- added C15, C16, C19, C20: 10nF, Capacitor_SMD:C_0603_1608Metric_Pad1.08x0.95mm_HandSolder, symbol Device:C
- added C3, C5: 120pF, Capacitor_SMD:C_0603_1608Metric_Pad1.08x0.95mm_HandSolder, symbol Device:C
- added C7, C8: 100nF, Capacitor_SMD:C_0603_1608Metric_Pad1.08x0.95mm_HandSolder, symbol Device:C
- added J5: Conn_Coaxial, symbol Connector:Conn_Coaxial
- added R10, R9: 3.3k, Resistor_SMD:R_0603_1608Metric_Pad0.98x0.95mm_HandSolder, symbol Device:R
- added R11: 2.32k, Resistor_SMD:R_0603_1608Metric_Pad0.98x0.95mm_HandSolder, symbol Device:R
- added R12: 7.15k, Resistor_SMD:R_0603_1608Metric_Pad0.98x0.95mm_HandSolder, symbol Device:R
- added R13: 1.74k, Resistor_SMD:R_0603_1608Metric_Pad0.98x0.95mm_HandSolder, symbol Device:R
- added R3: 1k, Resistor_SMD:R_0603_1608Metric_Pad0.98x0.95mm_HandSolder, symbol Device:R
- added R4, R5: 0R, Resistor_SMD:R_0603_1608Metric_Pad0.98x0.95mm_HandSolder, symbol Device:R
- added R6: 2.26k, Resistor_SMD:R_0603_1608Metric_Pad0.98x0.95mm_HandSolder, symbol Device:R
- added R7: 2.94k, Resistor_SMD:R_0603_1608Metric_Pad0.98x0.95mm_HandSolder, symbol Device:R
- added R8: 1.27k, Resistor_SMD:R_0603_1608Metric_Pad0.98x0.95mm_HandSolder, symbol Device:R
- added TP1, TP2, TP3, TP4, TP5, TP6: TP, TestPoint:TestPoint_Pad_D2.0mm, symbol Connector:TestPoint
- added U10: AD5252, Package_SO:TSSOP-14_4.4x5mm_P0.65mm, symbol own:AD5252
- added U11: LT1722, Package_TO_SOT_SMD:SOT-23-5_HandSoldering, symbol own:LT1722
- added U12: AD8039, Package_SO:SOIC-8_3.9x4.9mm_P1.27mm, symbol own:AD8039
- C2: renamed from C?; value C -> 1uF; footprint (none) -> Capacitor_SMD:C_0603_1608Metric_Pad1.08x0.95mm_HandSolder
- R1: renamed from R?; value R -> 50R; footprint (none) -> Resistor_SMD:R_0603_1608Metric_Pad0.98x0.95mm_HandSolder
- R2: renamed from R?; value R -> 22k; footprint (none) -> Resistor_SMD:R_0603_1608Metric_Pad0.98x0.95mm_HandSolder
Connections:
- net labels added: +2V5, -2V5, PGA_CTRL
- wire segments 66 -> 148
Other:
- note added: "AD8039 decoupling"
- note added: "Digipot decoupling"
- note added: "LT1722 decoupling"
- note removed: "Add buffer to match impedance?"
- moved on the sheet: C2, R1, R2

Commit message: Schematic finishing touches
Parts:
- added R14: 50R, symbol Device:R
- C1: value 1uF -> DNP
Connections:
- net IF_OUT: now also R14.1; no longer C12.1, R12.1, U12.7
- net SDA: now reaches R9.2, U10.7 (SDA)
- net SCL: now reaches R10.2, U10.9 (SCL)
- new net: C12.1, R12.1, R14.2, U12.7
Changed lines of the file:
@@
 $Descr A4 11693 8268
 encoding utf-8
-Sheet 2 5
+Sheet 2 6
 Title ""
 Date ""
@@
 $EndComp
 $Comp
-L power:GND #PWR0105
+L power:GND #PWR06
 U 1 1 5FA1EA1A
 P 3200 5900
-F 0 "#PWR0105" H 3200 5650 50  0001 C CNN
+F 0 "#PWR06" H 3200 5650 50  0001 C CNN
 F 1 "GND" H 3205 5727 50  0000 C CNN
 F 2 "" H 3200 5900 50  0001 C CNN
@@
 	3700 5450 3700 5550
 $Comp
-L power:GND #PWR0106
+L power:GND #PWR07
 U 1 1 5FA1FC7A
 P 3700 5900
-F 0 "#PWR0106" H 3700 5650 50  0001 C CNN
+F 0 "#PWR07" H 3700 5650 50  0001 C CNN
 F 1 "GND" H 3705 5727 50  0000 C CNN
 F 2 "" H 3700 5900 50  0001 C CNN
@@
 Wire Wire Line
 	3700 5850 3700 5900
-Text HLabel 9650 5750 2    100  Output ~ 0
+Text HLabel 10000 5750 2    100  Output ~ 0
 IF_OUT
 Wire Wire Line
@@
 	4700 5450 4200 5450
 $Comp
-L power:+2V5 #PWR0107
+L power:+2V5 #PWR013
 U 1 1 604CE4E3
 P 5000 5250
-F 0 "#PWR0107" H 5000 5100 50  0001 C CNN
+F 0 "#PWR013" H 5000 5100 50  0001 C CNN
 F 1 "+2V5" H 5015 5423 50  0000 C CNN
 F 2 "" H 5000 5250 50  0001 C CNN
@@
 	5000 5250 5000 5300
 $Comp
-L power:-2V5 #PWR0108
+L power:-2V5 #PWR014
 U 1 1 604CF877
 P 5000 5850
-F 0 "#PWR0108" H 5000 5950 50  0001 C CNN
+F 0 "#PWR014" H 5000 5950 50  0001 C CNN
 F 1 "-2V5" H 5015 6023 50  0000 C CNN
 F 2 "" H 5000 5850 50  0001 C CNN
@@
 	4900 4300 4900 4350
 $Comp
-L Device:R R4
-U 1 1 604D37EA
-P 4900 4500
-F 0 "R4" H 4750 4550 50  0000 L CNN
-F 1 "0R" H 4750 4450 50  0000 L CNN
-F 2 "Resistor_SMD:R_0603_1608Metric_Pad0.98x0.95mm_HandSolder" V 4830 4500 50  0001 C CNN
-F 3 "~" H 4900 4500 50  0001 C CNN
-	1    4900 4500
-	1    0    0    -1
-$EndComp
-$Comp
-L power:GND #PWR0109
+L power:GND #PWR012
 U 1 1 604D3D9F
 P 4900 4700
-F 0 "#PWR0109" H 4900 4450 50  0001 C CNN
+F 0 "#PWR012" H 4900 4450 50  0001 C CNN
 F 1 "GND" H 4905 4527 50  0000 C CNN
 F 2 "" H 4900 4700 50  0001 C CNN
@@
 	6600 5550 6750 5550
 $Comp
-L power:GND #PWR0110
+L power:GND #PWR021
 U 1 1 604DF486
 P 6850 5800
-F 0 "#PWR0110" H 6850 5550 50  0001 C CNN
+F 0 "#PWR021" H 6850 5550 50  0001 C CNN
 F 1 "GND" H 6855 5627 50  0000 C CNN
 F 2 "" H 6850 5800 50  0001 C CNN
@@
 Connection ~ 6750 5150
 $Comp
-L power:GND #PWR0111
+L power:GND #PWR018
 U 1 1 604E167C
 P 6250 5950
-F 0 "#PWR0111" H 6250 5700 50  0001 C CNN
+F 0 "#PWR018" H 6250 5700 50  0001 C CNN
 F 1 "GND" H 6255 5777 50  0000 C CNN
 F 2 "" H 6250 5950 50  0001 C CNN
@@
 	8000 5650 8000 5600
 $Comp
-L power:GND #PWR0112
+L power:GND #PWR025
 U 1 1 604E92E2
 P 8000 6050
-F 0 "#PWR0112" H 8000 5800 50  0001 C CNN
+F 0 "#PWR025" H 8000 5800 50  0001 C CNN
 F 1 "GND" H 8005 5877 50  0000 C CNN
 F 2 "" H 8000 6050 50  0001 C CNN
@@
 $EndComp
 $Comp
-L power:GND #PWR0113
+L power:GND #PWR027
 U 1 1 604E965B
 P 8600 5900
-F 0 "#PWR0113" H 8600 5650 50  0001 C CNN
+F 0 "#PWR027" H 8600 5650 50  0001 C CNN
 F 1 "GND" H 8605 5727 50  0000 C CNN
 F 2 "" H 8600 5900 50  0001 C CNN
@@
 	8500 5250 9300 5250
 Wire Wire Line
-	9300 5750 9650 5750
+	9300 5750 9450 5750
 Connection ~ 9300 5750
 $Comp
-L power:-2V5 #PWR0114
+L power:-2V5 #PWR011
 U 1 1 604EE3C5
 P 4400 4150
-F 0 "#PWR0114" H 4400 4250 50  0001 C CNN
+F 0 "#PWR011" H 4400 4250 50  0001 C CNN
 F 1 "-2V5" H 4415 4323 50  0000 C CNN
 F 2 "" H 4400 4150 50  0001 C CNN
@@
 	4400 4100 4400 4150
 $Comp
-L power:+2V5 #PWR0115
+L power:+2V5 #PWR010
 U 1 1 604EF8FE
 P 4400 3550
-F 0 "#PWR0115" H 4400 3400 50  0001 C CNN
+F 0 "#PWR010" H 4400 3400 50  0001 C CNN
 F 1 "+2V5" H 4415 3723 50  0000 C CNN
 F 2 "" H 4400 3550 50  0001 C CNN
@@
 $EndComp
 $Comp
-L power:GND #PWR0116
+L power:GND #PWR09
 U 1 1 605AD0A7
 P 4300 3900
-F 0 "#PWR0116" H 4300 3650 50  0001 C CNN
+F 0 "#PWR09" H 4300 3650 50  0001 C CNN
 F 1 "GND" H 4305 3727 50  0000 C CNN
 F 2 "" H 4300 3900 50  0001 C CNN
@@
 $EndComp
 $Comp
-L power:+2V5 #PWR0117
+L power:+2V5 #PWR017
 U 1 1 605B44E9
 P 6250 3550
-F 0 "#PWR0117" H 6250 3400 50  0001 C CNN
+F 0 "#PWR017" H 6250 3400 50  0001 C CNN
 F 1 "+2V5" H 6265 3723 50  0000 C CNN
 F 2 "" H 6250 3550 50  0001 C CNN
@@
 	5650 4350 5800 4350
 $Comp
-L power:GND #PWR0118
+L power:GND #PWR016
 U 1 1 605BD430
 P 5800 4400
-F 0 "#PWR0118" H 5800 4150 50  0001 C CNN
+F 0 "#PWR016" H 5800 4150 50  0001 C CNN
 F 1 "GND" H 5805 4227 50  0000 C CNN
 F 2 "" H 5800 4400 50  0001 C CNN
@@
 $EndComp
 $Comp
-L power:+2V5 #PWR0119
+L power:+2V5 #PWR032
 U 1 1 605C17FB
 P 10750 900
-F 0 "#PWR0119" H 10750 750 50  0001 C CNN
+F 0 "#PWR032" H 10750 750 50  0001 C CNN
 F 1 "+2V5" H 10765 1073 50  0000 C CNN
 F 2 "" H 10750 900 50  0001 C CNN
@@
 $EndComp
 $Comp
-L power:-2V5 #PWR0120
+L power:-2V5 #PWR033
 U 1 1 605C1FB4
 P 10750 2100
-F 0 "#PWR0120" H 10750 2200 50  0001 C CNN
+F 0 "#PWR033" H 10750 2200 50  0001 C CNN
 F 1 "-2V5" H 10765 2273 50  0000 C CNN
 F 2 "" H 10750 2100 50  0001 C CNN
@@
 	8900 2050 8900 2150
 $Comp
-L power:-2V5 #PWR0121
+L power:-2V5 #PWR029
 U 1 1 605EC19B
 P 8900 2150
-F 0 "#PWR0121" H 8900 2250 50  0001 C CNN
+F 0 "#PWR029" H 8900 2250 50  0001 C CNN
 F 1 "-2V5" H 8915 2323 50  0000 C CNN
 F 2 "" H 8900 2150 50  0001 C CNN
@@
 	8900 900  8900 1000
 $Comp
-L power:+2V5 #PWR0122
+L power:+2V5 #PWR028
 U 1 1 605EEF1E
 P 8900 900
-F 0 "#PWR0122" H 8900 750 50  0001 C CNN
+F 0 "#PWR028" H 8900 750 50  0001 C CNN
 F 1 "+2V5" H 8915 1073 50  0000 C CNN
 F 2 "" H 8900 900 50  0001 C CNN
@@
 	9300 1500 9300 1600
 $Comp
-L power:GND #PWR0123
+L power:GND #PWR030
 U 1 1 6062C0F2
 P 9300 1600
-F 0 "#PWR0123" H 9300 1350 50  0001 C CNN
+F 0 "#PWR030" H 9300 1350 50  0001 C CNN
 F 1 "GND" H 9305 1427 50  0000 C CNN
 F 2 "" H 9300 1600 50  0001 C CNN
@@
 Connection ~ 10350 1500
 $Comp
-L power:GND #PWR0124
+L power:GND #PWR031
 U 1 1 606678E6
 P 9750 1600
-F 0 "#PWR0124" H 9750 1350 50  0001 C CNN
+F 0 "#PWR031" H 9750 1350 50  0001 C CNN
 F 1 "GND" H 9755 1427 50  0000 C CNN
 F 2 "" H 9750 1600 50  0001 C CNN
@@
 Wire Wire Line
 	9750 1500 9750 1600
-Entry Wire Line
-	7050 3950 7150 3850
-Entry Wire Line
-	7050 4050 7150 3950
-Text HLabel 7150 3750 1    50   BiDi ~ 0
-PGA_CTRL
 Wire Wire Line
 	6200 3950 6500 3950
@@
 	6200 4050 6800 4050
 $Comp
-L power:+2V5 #PWR0125
+L power:+2V5 #PWR019
 U 1 1 6069E916
 P 6500 3450
-F 0 "#PWR0125" H 6500 3300 50  0001 C CNN
+F 0 "#PWR019" H 6500 3300 50  0001 C CNN
 F 1 "+2V5" H 6515 3623 50  0000 C CNN
 F 2 "" H 6500 3450 50  0001 C CNN
@@
 $EndComp
 $Comp
-L power:+2V5 #PWR0126
+L power:+2V5 #PWR020
 U 1 1 6069EB38
 P 6800 3450
-F 0 "#PWR0126" H 6800 3300 50  0001 C CNN
+F 0 "#PWR020" H 6800 3300 50  0001 C CNN
 F 1 "+2V5" H 6815 3623 50  0000 C CNN
 F 2 "" H 6800 3450 50  0001 C CNN
@@
 	7750 2050 7750 2150
 $Comp
-L power:-2V5 #PWR0127
+L power:-2V5 #PWR024
 U 1 1 606B7D7B
 P 7750 2150
-F 0 "#PWR0127" H 7750 2250 50  0001 C CNN
+F 0 "#PWR024" H 7750 2250 50  0001 C CNN
 F 1 "-2V5" H 7765 2323 50  0000 C CNN
 F 2 "" H 7750 2150 50  0001 C CNN
@@
 	7750 900  7750 1000
 $Comp
-L power:+2V5 #PWR0128
+L power:+2V5 #PWR023
 U 1 1 606B7D95
 P 7750 900
-F 0 "#PWR0128" H 7750 750 50  0001 C CNN
+F 0 "#PWR023" H 7750 750 50  0001 C CNN
 F 1 "+2V5" H 7765 1073 50  0000 C CNN
 F 2 "" H 7750 900 50  0001 C CNN
@@
 	8150 1500 8150 1600
 $Comp
-L power:GND #PWR0129
+L power:GND #PWR026
 U 1 1 606B7DA1
 P 8150 1600
-F 0 "#PWR0129" H 8150 1350 50  0001 C CNN
+F 0 "#PWR026" H 8150 1350 50  0001 C CNN
 F 1 "GND" H 8155 1427 50  0000 C CNN
 F 2 "" H 8150 1600 50  0001 C CNN
@@
 	5450 5550 5450 5650
 $Comp
-L power:GND #PWR0131
+L power:GND #PWR015
 U 1 1 6082EC77
 P 5450 6150
-F 0 "#PWR0131" H 5450 5900 50  0001 C CNN
+F 0 "#PWR015" H 5450 5900 50  0001 C CNN
 F 1 "GND" H 5455 5977 50  0000 C CNN
 F 2 "" H 5450 6150 50  0001 C CNN
@@
 	5450 6150 5450 6050
 $Comp
-L power:GND #PWR0132
+L power:GND #PWR022
 U 1 1 60837F8E
 P 7550 6250
-F 0 "#PWR0132" H 7550 6000 50  0001 C CNN
+F 0 "#PWR022" H 7550 6000 50  0001 C CNN
 F 1 "GND" H 7555 6077 50  0000 C CNN
 F 2 "" H 7550 6250 50  0001 C CNN
@@
 AR Path="/605249CC/60855A76" Ref="C1"  Part="1"
 F 0 "C1" V 2948 5200 50  0000 C CNN
-F 1 "1uF" V 3039 5200 50  0000 C CNN
+F 1 "DNP" V 3039 5200 50  0000 C CNN
 F 2 "Capacitor_SMD:C_0603_1608Metric_Pad1.08x0.95mm_HandSolder" H 3238 5050 50  0001 C CNN
 F 3 "~" H 3200 5200 50  0001 C CNN
@@
 P 2950 4750
 AR Path="/60524BC3/60855A82" Ref="#PWR?"  Part="1"
-AR Path="/605249CC/60855A82" Ref="#PWR0133"  Part="1"
-F 0 "#PWR0133" H 2950 4500 50  0001 C CNN
+AR Path="/605249CC/60855A82" Ref="#PWR05"  Part="1"
+F 0 "#PWR05" H 2950 4500 50  0001 C CNN
 F 1 "GND" H 2955 4577 50  0000 C CNN
 F 2 "" H 2950 4750 50  0001 C CNN
@@
 	4200 5950 4200 6050
 $Comp
-L power:GND #PWR0130
+L power:GND #PWR08
 U 1 1 608155B7
 P 4200 6050
-F 0 "#PWR0130" H 4200 5800 50  0001 C CNN
+F 0 "#PWR08" H 4200 5800 50  0001 C CNN
 F 1 "GND" H 4205 5877 50  0000 C CNN
 F 2 "" H 4200 6050 50  0001 C CNN
@@
 	1    0    0    -1
 $EndComp
-Wire Bus Line
-	7150 3750 7150 3950
+$Comp
+L Device:R R4
+U 1 1 604D37EA
+P 4900 4500
+F 0 "R4" H 4750 4550 50  0000 L CNN
+F 1 "0R" H 4750 4450 50  0000 L CNN
+F 2 "Resistor_SMD:R_0603_1608Metric_Pad0.98x0.95mm_HandSolder" V 4830 4500 50  0001 C CNN
+F 3 "~" H 4900 4500 50  0001 C CNN
+	1    4900 4500
+	1    0    0    -1
+$EndComp
+$Comp
+L Device:R R14
+U 1 1 606069A9
+P 9600 5750
+F 0 "R14" V 9393 5750 50  0000 C CNN
+F 1 "50R" V 9484 5750 50  0000 C CNN
+F 2 "" V 9530 5750 50  0001 C CNN
+F 3 "~" H 9600 5750 50  0001 C CNN
+	1    9600 5750
+	0    1    1    0
+$EndComp
+Wire Wire Line
+	9750 5750 10000 5750
+Text Label 6600 3950 0    50   ~ 0
+SDA
+Text Label 6600 4050 0    50   ~ 0
+SCL
+Text HLabel 7050 3950 2    50   BiDi ~ 0
+SDA
+Text HLabel 7050 4050 2    50   Input ~ 0
+SCL
 $EndSCHEMATC

Commit message: First layout
Parts:
- J5: footprint (none) -> Connector_Coaxial:SMA_Amphenol_901-144_Vertical
- R14: footprint (none) -> Resistor_SMD:R_0603_1608Metric_Pad0.98x0.95mm_HandSolder
Changed lines of the file:
@@
 F 0 "J5" V 3437 4629 50  0000 C CNN
 F 1 "Conn_Coaxial" V 3346 4629 50  0000 C CNN
-F 2 "" H 3200 4700 50  0001 C CNN
+F 2 "Connector_Coaxial:SMA_Amphenol_901-144_Vertical" H 3200 4700 50  0001 C CNN
 F 3 " ~" H 3200 4700 50  0001 C CNN
 	1    3200 4700
@@
 F 0 "R14" V 9393 5750 50  0000 C CNN
 F 1 "50R" V 9484 5750 50  0000 C CNN
-F 2 "" V 9530 5750 50  0001 C CNN
+F 2 "Resistor_SMD:R_0603_1608Metric_Pad0.98x0.95mm_HandSolder" V 9530 5750 50  0001 C CNN
 F 3 "~" H 9600 5750 50  0001 C CNN
 	1    9600 5750

Commit message: IF and power layout mostly finished
Parts:
- removed TP4: TP, TestPoint:TestPoint_Pad_D2.0mm, symbol Connector:TestPoint
- J5: footprint Connector_Coaxial:SMA_Amphenol_901-144_Vertical -> Connector_Coaxial:SMA_Amphenol_132134-11_Vertical
Changed lines of the file:
@@
 	4400 3600 4400 3550
-$Comp
-L own:AD5252 U10
-U 1 1 605A5EA2
-P 4850 4000
-F 0 "U10" H 5325 4665 50  0000 C CNN
-F 1 "AD5252" H 5325 4574 50  0000 C CNN
-F 2 "Package_SO:TSSOP-14_4.4x5mm_P0.65mm" H 4250 3450 50  0001 C CNN
-F 3 "" H 4250 3450 50  0001 C CNN
-	1    4850 4000
-	1    0    0    -1
-$EndComp
 $Comp
 L power:GND #PWR09
@@
 Wire Wire Line
 	5450 5550 5450 5650
-$Comp
-L power:GND #PWR015
-U 1 1 6082EC77
-P 5450 6150
-F 0 "#PWR015" H 5450 5900 50  0001 C CNN
-F 1 "GND" H 5455 5977 50  0000 C CNN
-F 2 "" H 5450 6150 50  0001 C CNN
-F 3 "" H 5450 6150 50  0001 C CNN
-	1    5450 6150
-	1    0    0    -1
-$EndComp
-Wire Wire Line
-	5450 6150 5450 6050
 $Comp
 L power:GND #PWR022
@@
 F 0 "J5" V 3437 4629 50  0000 C CNN
 F 1 "Conn_Coaxial" V 3346 4629 50  0000 C CNN
-F 2 "Connector_Coaxial:SMA_Amphenol_901-144_Vertical" H 3200 4700 50  0001 C CNN
+F 2 "Connector_Coaxial:SMA_Amphenol_132134-11_Vertical" H 3200 4700 50  0001 C CNN
 F 3 " ~" H 3200 4700 50  0001 C CNN
 	1    3200 4700
@@
 $EndComp
 $Comp
-L Connector:TestPoint TP4
-U 1 1 609439EE
-P 5450 6050
-F 0 "TP4" H 5508 6168 50  0000 L CNN
-F 1 "TP" H 5508 6077 50  0000 L CNN
-F 2 "TestPoint:TestPoint_Pad_D2.0mm" H 5650 6050 50  0001 C CNN
-F 3 "~" H 5650 6050 50  0001 C CNN
-	1    5450 6050
-	1    0    0    -1
-$EndComp
-$Comp
 L Connector:TestPoint TP5
 U 1 1 609500A3
@@
 Text HLabel 7050 4050 2    50   Input ~ 0
 SCL
+$Comp
+L own:AD5252 U10
+U 1 1 605A5EA2
+P 4850 4000
+F 0 "U10" H 5325 4665 50  0000 C CNN
+F 1 "AD5252" H 5325 4574 50  0000 C CNN
+F 2 "Package_SO:TSSOP-14_4.4x5mm_P0.65mm" H 4250 3450 50  0001 C CNN
+F 3 "" H 4250 3450 50  0001 C CNN
+	1    4850 4000
+	1    0    0    -1
+$EndComp
 $EndSCHEMATC
